Commit message: removed absolute paths, replaced with relative

File: src/jackal_description/urdf/jackal.urdf.xacro (robot description, xacro)
@@ -219,5 +219,5 @@
   </joint>
   <!--add my 2d lidar to the chassis. -->
-  <xacro:include filename="/home/jidan/Documents/Autonomous_Mobile_Robotics/ME5413_Final_Project/src/jackal_description/urdf/lidar_gazebo.xacro" />
+  <xacro:include filename="$(find jackal_description)/urdf/lidar_gazebo.xacro" />
   <xacro:rplidar prefix="laser"/>
   <joint name="lidar_joint" type="fixed">
@@ -226,5 +226,5 @@
     <origin xyz="0 0 -0.209" />
   </joint>
-  <xacro:include filename="/home/jidan/Documents/Autonomous_Mobile_Robotics/ME5413_Final_Project/src/jackal_description/urdf/kinect_gazebo.xacro" />
+  <xacro:include filename="$(find jackal_description)/urdf/kinect_gazebo.xacro" />
   <xacro:kinect_camera prefix="kinect"/>
   <joint name="kinect_joint" type="fixed">

File: src/jackal_description/urdf/kinect_gazebo.xacro (robot description, xacro)
@@ -9,5 +9,5 @@
                 <origin xyz="0 0 0" rpy="0 0 ${3.14/2}"/>
                 <geometry>
-                    <mesh filename="/home/jidan/Documents/Autonomous_Mobile_Robotics/ME5413_Final_Project/src/jackal_description/urdf/meshes/kinect.dae" />
+                    <mesh filename="$(find jackal_description)/urdf/meshes/kinect.dae" />
                 </geometry>
             </visual>
