Commit message: feat: updated jackal_description

File: src/jackal_description/urdf/accessories.urdf.xacro (robot description, xacro)
@@ -46,5 +46,5 @@
   -->
   <!-- Primary 2D Lidar -->
-  <xacro:if value="$(optenv JACKAL_LASER 1)">
+  <xacro:if value="$(optenv JACKAL_LASER 0)">
     <xacro:property name="mount" value="$(optenv JACKAL_LASER_MOUNT front)" />
     <xacro:property name="topic" value="$(optenv JACKAL_LASER_TOPIC front/scan)" />
@@ -169,5 +169,5 @@
     - vlp32e           :: Velodyne HDL-32E
   -->
-  <xacro:if value="$(optenv JACKAL_LASER_3D 1)">
+  <xacro:if value="$(optenv JACKAL_LASER_3D 0)">
     <xacro:property name="mount" value="$(optenv JACKAL_LASER_3D_MOUNT mid)" />
     <xacro:property name="topic" value="$(optenv JACKAL_LASER_3D_TOPIC mid/points)" />
@@ -260,5 +260,5 @@
   <xacro:include filename="$(find pointgrey_camera_description)/urdf/pointgrey_flea3.urdf.xacro" />
   <!-- If enabled, generate the flea3 camera payload with a tilt of 30 degrees. -->
-  <xacro:if value="$(optenv JACKAL_FLEA3 1)">
+  <xacro:if value="$(optenv JACKAL_FLEA3 0)">
     <xacro:property name="name" value="$(optenv JACKAL_FLEA3_NAME front)" />
     <xacro:property name="tilt" value="$(optenv JACKAL_FLEA3_TILT 0.)" />

File: src/jackal_description/urdf/jackal.urdf.xacro (robot description, xacro)
@@ -218,4 +218,19 @@
     <origin xyz="${mount_spacing} 0 0" />
   </joint>
+  <!--add my 2d lidar to the chassis. -->
+  <xacro:include filename="/home/jidan/Documents/Autonomous_Mobile_Robotics/ME5413_Final_Project/src/jackal_description/urdf/lidar_gazebo.xacro" />
+  <xacro:rplidar prefix="laser"/>
+  <joint name="lidar_joint" type="fixed">
+    <parent link="mid_mount" />
+    <child link="laser_link" />
+    <origin xyz="0 0 -0.209" />
+  </joint>
+  <xacro:include filename="/home/jidan/Documents/Autonomous_Mobile_Robotics/ME5413_Final_Project/src/jackal_description/urdf/kinect_gazebo.xacro" />
+  <xacro:kinect_camera prefix="kinect"/>
+  <joint name="kinect_joint" type="fixed">
+    <parent link="mid_mount" />
+    <child link="kinect_link" />
+    <origin xyz="0.15 0 0.035" />
+  </joint>
   <!-- Bring in simulation data for Gazebo. -->
   <xacro:include filename="$(find jackal_description)/urdf/jackal.gazebo" />

Commit message: feat: updated models

File: src/jackal_description/urdf/accessories.urdf.xacro (robot description, xacro)
@@ -46,5 +46,5 @@
   -->
   <!-- Primary 2D Lidar -->
-  <xacro:if value="$(optenv JACKAL_LASER 0)">
+  <xacro:if value="$(optenv JACKAL_LASER 1)">
     <xacro:property name="mount" value="$(optenv JACKAL_LASER_MOUNT front)" />
     <xacro:property name="topic" value="$(optenv JACKAL_LASER_TOPIC front/scan)" />
@@ -52,5 +52,5 @@
     <xacro:property name="prefix" value="$(optenv JACKAL_LASER_PREFIX ${mount})" />
     <xacro:property name="parent" value="$(optenv JACKAL_LASER_PARENT ${mount}_mount)" />
-    <xacro:property name="lidar_model" value="$(optenv JACKAL_LASER_MODEL tim551)" />
+    <xacro:property name="lidar_model" value="$(optenv JACKAL_LASER_MODEL lms1xx)" />
     <xacro:property name="mount_type" value="$(optenv JACKAL_LASER_MOUNT_TYPE upright)" />
     <!-- SICK LMS1xx -->
@@ -60,5 +60,5 @@
         <xacro:if value="${mount_type == 'upright'}">
           <xacro:sick_lms1xx_upright_mount topic="${topic}" prefix="${prefix}" parent_link="${parent}">
-            <origin xyz="$(optenv JACKAL_LASER_OFFSET 0 0 0)" rpy="$(optenv JACKAL_LASER_RPY 0 0 0)" />
+            <origin xyz="$(optenv JACKAL_LASER_OFFSET -0.12 0 0.16)" rpy="$(optenv JACKAL_LASER_RPY 0 0 0)" />
           </xacro:sick_lms1xx_upright_mount>
         </xacro:if>
@@ -172,8 +172,8 @@
     <xacro:property name="mount" value="$(optenv JACKAL_LASER_3D_MOUNT mid)" />
     <xacro:property name="topic" value="$(optenv JACKAL_LASER_3D_TOPIC mid/points)" />
-    <xacro:property name="tower" value="$(optenv JACKAL_LASER_3D_TOWER 1)" />
+    <xacro:property name="tower" value="$(optenv JACKAL_LASER_3D_TOWER 0)" />
     <xacro:property name="prefix" value="$(optenv JACKAL_LASER_3D_PREFIX ${mount})" />
     <xacro:property name="parent" value="$(optenv JACKAL_LASER_3D_PARENT ${mount}_mount)" />
-    <xacro:property name="lidar_3d_model" value="$(optenv JACKAL_LASER_3D_MODEL vlp16)" />
+    <xacro:property name="lidar_3d_model" value="$(optenv JACKAL_LASER_3D_MODEL hdl32e)" />
     <!-- Velodyne VLP16 -->
     <xacro:if value="${lidar_3d_model == 'vlp16'}">
@@ -185,5 +185,5 @@
     <xacro:if value="${lidar_3d_model == 'hdl32e'}">
       <xacro:hdl32e_mount topic="${topic}" tower="${tower}" prefix="${prefix}" parent_link="${parent}" >
-        <origin xyz="$(optenv JACKAL_LASER_3D_OFFSET 0 0 0)" rpy="$(optenv JACKAL_LASER_3D_RPY 0 0 0)" />
+        <origin xyz="$(optenv JACKAL_LASER_3D_OFFSET 0 0 0.7)" rpy="$(optenv JACKAL_LASER_3D_RPY 0 0 0)" />
       </xacro:hdl32e_mount>
     </xacro:if>

File: src/jackal_description/urdf/accessories/hdl32_mount.urdf.xacro (robot description, xacro)
@@ -29,5 +29,28 @@
     </xacro:if>
     <xacro:unless value="${tower}">
-      <link name="${prefix}_hdl32e_mount"/>
+      <!--modify version_add the height of the velodyne-->
+      <link name="${prefix}_hdl32e_mount">
+        <visual>
+          <geometry>
+            <cylinder radius="0.04" length = "1.4"/>
+          </geometry>
+          <origin xyz="0 0 0" rpy="0 0 0" />
+          <material name="black" />
+        </visual>
+        <collision>
+          <geometry>
+            <cylinder radius="0.04" length = "1.4"/>
+          </geometry>
+          <origin xyz="0 0 0" rpy="0 0 0" />
+        </collision>
+        <inertial>
+          <origin xyz="0 0 0" rpy="0 0 0"/>
+          <mass value="0.2"/>
+          <inertia
+            ixx="0.032746667" ixy="0" ixz="0"
+            iyy="0.032746667" iyz="0"
+            izz="0.00016"/>
+        </inertial>
+      </link>
       <joint name="${prefix}_hdl32e_mount_joint" type="fixed">
         <parent link="${parent_link}"/>
@@ -37,5 +60,6 @@
       <!-- Velodyne HDL-32E Macro treats Y-axis as forward in pointcloud -->
       <xacro:HDL-32E parent="${prefix}_hdl32e_mount" topic="${topic}">
-        <origin xyz="0 0 0" rpy="0 0 -1.5707"/>
+        <!--origin xyz="0 0 0" rpy="0 0 -1.5707"-->
+        <origin xyz="0 0 0.7" rpy="0 0 -1.5707"/>
       </xacro:HDL-32E>
     </xacro:unless>

File: src/jackal_description/urdf/jackal.urdf.xacro (robot description, xacro)
@@ -226,5 +226,5 @@
     <origin xyz="0 0 -0.209" />
   </joint>
-  <!--add my camera to the chassis.
+  <!--add my camera to the chassis. -->
   <xacro:include filename="$(find jackal_description)/urdf/kinect_gazebo.xacro" />
   <xacro:kinect_camera prefix="kinect"/>
@@ -234,5 +234,4 @@
     <origin xyz="0.15 0 0.035" />
   </joint>
--->
   <!-- Bring in simulation data for Gazebo. -->
   <xacro:include filename="$(find jackal_description)/urdf/jackal.gazebo" />

File: src/jackal_description/urdf/kinect_gazebo.xacro (robot description, xacro)
@@ -9,5 +9,5 @@
                 <origin xyz="0 0 0" rpy="0 0 ${3.14/2}"/>
                 <geometry>
-                    <mesh filename="$(find jackal_description)/urdf/meshes/kinect.dae" />
+                    <mesh filename="package://jackal_description/urdf/meshes/kinect.dae" />
                 </geometry>
             </visual>

Commit message: feat: updated models

File: src/jackal_description/urdf/accessories.urdf.xacro (robot description, xacro)
@@ -46,5 +46,5 @@
   -->
   <!-- Primary 2D Lidar -->
-  <xacro:if value="$(optenv JACKAL_LASER 1)">
+  <xacro:if value="$(optenv JACKAL_LASER 0)">
     <xacro:property name="mount" value="$(optenv JACKAL_LASER_MOUNT front)" />
     <xacro:property name="topic" value="$(optenv JACKAL_LASER_TOPIC front/scan)" />
@@ -60,5 +60,5 @@
         <xacro:if value="${mount_type == 'upright'}">
           <xacro:sick_lms1xx_upright_mount topic="${topic}" prefix="${prefix}" parent_link="${parent}">
-            <origin xyz="$(optenv JACKAL_LASER_OFFSET -0.12 0 0.16)" rpy="$(optenv JACKAL_LASER_RPY 0 0 0)" />
+            <origin xyz="$(optenv JACKAL_LASER_OFFSET -0.12 0 0)" rpy="$(optenv JACKAL_LASER_RPY 0 0 0)" />
           </xacro:sick_lms1xx_upright_mount>
         </xacro:if>
@@ -169,5 +169,5 @@
     - vlp32e           :: Velodyne HDL-32E
   -->
-  <xacro:if value="$(optenv JACKAL_LASER_3D 0)">
+  <xacro:if value="$(optenv JACKAL_LASER_3D 1)">
     <xacro:property name="mount" value="$(optenv JACKAL_LASER_3D_MOUNT mid)" />
     <xacro:property name="topic" value="$(optenv JACKAL_LASER_3D_TOPIC mid/points)" />

File: src/jackal_description/urdf/jackal.urdf.xacro (robot description, xacro)
@@ -218,5 +218,5 @@
     <origin xyz="${mount_spacing} 0 0" />
   </joint>
-  <!--add my 2d lidar to the chassis. -->
+  <!--add my 2d lidar to the chassis.
   <xacro:include filename="$(find jackal_description)/urdf/lidar_gazebo.xacro" />
   <xacro:rplidar prefix="laser"/>
@@ -225,6 +225,6 @@
     <child link="laser_link" />
     <origin xyz="0 0 -0.209" />
-  </joint>
-  <!--add my camera to the chassis. -->
+  </joint>-->
+  <!--add my camera to the chassis.
   <xacro:include filename="$(find jackal_description)/urdf/kinect_gazebo.xacro" />
   <xacro:kinect_camera prefix="kinect"/>
@@ -233,5 +233,5 @@
     <child link="kinect_link" />
     <origin xyz="0.15 0 0.035" />
-  </joint>
+  </joint>-->
   <!-- Bring in simulation data for Gazebo. -->
   <xacro:include filename="$(find jackal_description)/urdf/jackal.gazebo" />
